Commit message: added multi camera calibration tab and changed ui

File: pybullet_sim/urdf/gantry.urdf (robot description, URDF)
Before this commit: robot pod_farm_gantry, 19 links, 18 joints
Links:
- link back_camera_stage_link: geometry visual box size=0.03 0.018 0.03; visual box size=0.03 0.018 0.03
- link front_camera_stage_link: geometry visual box size=0.03 0.018 0.03; visual box size=0.03 0.018 0.03
